File: basic-lipo-manager.brd (EAGLE design)
At the start: 52.1 x 14 mm, 24 parts, among them U2 MCP73831

Commit message: label edits, fiducials added
Parts:
- added FID1, FID2, FID3: FIDUCIAL1X2, SparkFun-Aesthetics:FIDUCIAL-1X2
- moved U$4 7.64 mm to (40.9, 10.2)
- moved U$7 1.61 mm to (25.4, 2.79)
Routing:
- net VREG_IN: track 42.9 -> 44.1 mm
Other:
- board text added: "3V3"
- board text added: "AWQUA basic lipo manager 2017-09-15 v1.0 CDK"
- board text added: "OFF"
- board text added: "ON"
- board text added: "VDD"
- board text removed: "AWQUA basic lipo board 2017-09-15 v1.0 CDK"
Changed lines of the file:
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@@
 <board>
 <plain>
-<text x="38.5762" y="8.6995" size="0.8128" layer="21">AWQUA
-basic lipo board
+<text x="37.8142" y="0.3175" size="0.8128" layer="21">AWQUA
+basic lipo
+manager
 2017-09-15
 v1.0 CDK</text>
@@
 <wire x1="0.915809375" y1="13.97" x2="0" y2="13.054190625" width="0.254" layer="20" curve="90"/>
 <text x="30.48" y="-9.144" size="1.778" layer="25">AWQUA</text>
+<text x="21.8122" y="12.0015" size="1.524" layer="21">ON</text>
+<text x="21.0502" y="0.0635" size="1.524" layer="21">OFF</text>
+<text x="46.7042" y="11.2395" size="1.524" layer="21">3V3</text>
+<text x="0.7302" y="11.2395" size="1.524" layer="21">VDD</text>
 </plain>
 <attributes>
@@
 </element>
 <element name="FRAME1" library="SparkFun-Aesthetics" package="CREATIVE_COMMONS" value="FRAME-LETTER" x="-0.635" y="-8.89"/>
-<element name="U$4" library="SparkFun-Aesthetics" package="OSHW-LOGO-M" value="" x="43.688" y="3.048"/>
+<element name="U$4" library="SparkFun-Aesthetics" package="OSHW-LOGO-M" value="" x="40.894" y="10.16"/>
 <element name="D1" library="SparkFun" package="LED-0603" value="RED" x="33.528" y="7.112" rot="R90"/>
 <element name="R3" library="SparkFun" package="0402-RES" value="330" x="36.576" y="7.112"/>
@@
 <element name="D2" library="SparkFun" package="LED-0603" value="GRN" x="27.178" y="7.112" rot="R90"/>
 <element name="U$3" library="awqua_eagle_library" package="USBMICRO-10118193-0001LF" value="USBMICRO-10118193-0001LF" x="31.242" y="0.254"/>
-<element name="U$7" library="awqua_eagle_library" package="OS102-SPDT-SWITCH" value="OS102-SPDT-SWITCH" x="24.892" y="1.27" rot="R90"/>
+<element name="U$7" library="awqua_eagle_library" package="OS102-SPDT-SWITCH" value="OS102-SPDT-SWITCH" x="25.4" y="2.794" rot="R90"/>
 <element name="JP1" library="SparkFun-Connectors" package="1X04" value="" x="1.27" y="1.27" smashed="yes" rot="R90">
 <attribute name="VALUE" x="4.445" y="0" size="1.27" layer="27" rot="R90"/>
@@
 <attribute name="VALUE" x="13.462" y="15.875" size="1.27" layer="27" rot="R180"/>
 </element>
+<element name="FID1" library="SparkFun-Aesthetics" package="FIDUCIAL-1X2" value="FIDUCIAL1X2" x="6.35" y="9.652"/>
+<element name="FID2" library="SparkFun-Aesthetics" package="FIDUCIAL-1X2" value="FIDUCIAL1X2" x="36.83" y="4.826"/>
+<element name="FID3" library="SparkFun-Aesthetics" package="FIDUCIAL-1X2" value="FIDUCIAL1X2" x="44.45" y="12.446"/>
 </elements>
 <signals>
@@
 <wire x1="42.672" y1="6.35" x2="39.878" y2="3.556" width="0.4064" layer="16"/>
 <wire x1="39.878" y1="3.556" x2="26.162" y2="3.556" width="0.4064" layer="16"/>
-<wire x1="26.162" y1="3.556" x2="24.638" y2="5.08" width="0.4064" layer="16"/>
-<via x="24.638" y="5.08" extent="1-16" drill="0.3302"/>
-<wire x1="24.638" y1="5.08" x2="24.638" y2="8.128" width="0.4064" layer="1"/>
-<wire x1="24.638" y1="8.128" x2="24.638" y2="10.668" width="0.254" layer="1"/>
+<wire x1="26.162" y1="3.556" x2="24.638" y2="5.08" width="0.4064" layer="1"/>
+<wire x1="24.638" y1="5.08" x2="24.638" y2="10.668" width="0.4064" layer="1"/>
 <wire x1="24.638" y1="10.668" x2="23.876" y2="11.43" width="0.254" layer="1"/>
 <wire x1="23.876" y1="11.43" x2="18.034" y2="11.43" width="0.254" layer="1"/>
@@
 <wire x1="48.26" y1="6.35" x2="48.26" y2="3.81" width="0.4064" layer="16"/>
 <wire x1="48.26" y1="3.81" x2="48.26" y2="1.27" width="0.4064" layer="1"/>
+<via x="26.162" y="3.556" extent="1-16" drill="0.3302"/>
 </signal>
 <signal name="VOLT">
@@
 <wire x1="31.6539" y1="9.398" x2="31.7199" y2="9.464" width="0.254" layer="1"/>
 <contactref element="U$7" pad="P$3"/>
-<wire x1="22.742" y1="7.57" x2="22.91" y2="7.62" width="0.254" layer="16"/>
-<wire x1="22.91" y1="7.62" x2="25.908" y2="7.62" width="0.254" layer="16"/>
-<wire x1="25.908" y1="7.62" x2="25.908" y2="9.144" width="0.254" layer="16"/>
-<via x="25.908" y="9.144" extent="1-16" drill="0.3302"/>
-<wire x1="25.908" y1="9.144" x2="27.432" y2="9.144" width="0.254" layer="1"/>
+<wire x1="23.25" y1="9.094" x2="22.91" y2="9.144" width="0.254" layer="16"/>
+<wire x1="22.91" y1="9.144" x2="26.416" y2="9.144" width="0.254" layer="16"/>
+<via x="26.416" y="9.144" extent="1-16" drill="0.3302"/>
+<wire x1="26.416" y1="9.144" x2="27.432" y2="9.144" width="0.254" layer="1"/>
 <wire x1="27.432" y1="9.144" x2="27.94" y2="9.256" width="0.254" layer="1"/>
 <wire x1="9.922" y1="7.764" x2="9.922" y2="4.81" width="0.254" layer="1"/>
@@
 <wire x1="10.16" y1="4.572" x2="12.954" y2="4.572" width="0.254" layer="16"/>
 <wire x1="12.954" y1="4.572" x2="14.732" y2="6.35" width="0.254" layer="16"/>
-<wire x1="14.732" y1="6.35" x2="20.066" y2="6.35" width="0.254" layer="16"/>
-<wire x1="20.066" y1="6.35" x2="21.336" y2="7.62" width="0.254" layer="16"/>
-<wire x1="21.336" y1="7.62" x2="22.692" y2="7.62" width="0.254" layer="16"/>
-<wire x1="22.692" y1="7.62" x2="22.742" y2="7.57" width="0.254" layer="16"/>
+<wire x1="14.732" y1="6.35" x2="19.558" y2="6.35" width="0.254" layer="16"/>
+<wire x1="19.558" y1="6.35" x2="21.336" y2="8.128" width="0.254" layer="16"/>
+<wire x1="21.336" y1="8.128" x2="21.336" y2="8.382" width="0.254" layer="16"/>
+<wire x1="21.336" y1="8.382" x2="22.098" y2="9.144" width="0.254" layer="16"/>
+<wire x1="22.098" y1="9.144" x2="22.692" y2="9.144" width="0.254" layer="16"/>
+<wire x1="22.692" y1="9.144" x2="23.25" y2="9.094" width="0.254" layer="16"/>
 </signal>
 <signal name="VREG_IN">
@@
 <wire x1="19.05" y1="4.826" x2="19.05" y2="3.8459" width="0.254" layer="1"/>
 <wire x1="19.05" y1="3.8459" x2="18.984" y2="3.7799" width="0.254" layer="1"/>
-<wire x1="20.32" y1="4.826" x2="19.05" y2="4.826" width="0.254" layer="1"/>
+<wire x1="20.828" y1="4.826" x2="19.05" y2="4.826" width="0.254" layer="1"/>
 <contactref element="JP1" pad="1"/>
 <contactref element="JP1" pad="2"/>
 <contactref element="JP1" pad="3"/>
 <contactref element="JP1" pad="4"/>
-<wire x1="20.32" y1="4.826" x2="20.32" y2="5.316" width="0.254" layer="1"/>
-<wire x1="20.32" y1="5.316" x2="20.574" y2="5.57" width="0.254" layer="1"/>
-<wire x1="20.574" y1="5.57" x2="22.742" y2="5.57" width="0.254" layer="1"/>
+<wire x1="20.828" y1="4.826" x2="20.828" y2="5.316" width="0.254" layer="1"/>
+<wire x1="20.828" y1="5.316" x2="22.606" y2="7.094" width="0.254" layer="1"/>
+<wire x1="22.606" y1="7.094" x2="23.25" y2="7.094" width="0.254" layer="1"/>
 <wire x1="16.09" y1="12.192" x2="16.09" y2="11.518" width="0.254" layer="1"/>
 <wire x1="16.09" y1="11.518" x2="15.494" y2="10.922" width="0.254" layer="1"/>
